Commit message: added filed to allow simulation of 2 UR5s

File: ur_description/urdf/ur5_double_limited.urdf.xacro (robot description, xacro)
@@ -1,5 +1,5 @@
 <?xml version="1.0"?>
 <robot xmlns:xacro="http://ros.org/wiki/xacro"
-       name="ur5_robotiq85_kinect" >
+       name="ur5_double" >
   <!-- common stuff -->
   <xacro:include filename="$(find ur_description)/urdf/common.gazebo.xacro" />
@@ -7,7 +7,7 @@
   <xacro:include filename="$(find ur_description)/urdf/ur5.urdf.xacro" />
   <!-- left arm -->
-  <xacro:ur5_robot prefix="left_" joint_limited="false"/>
+  <xacro:ur5_robot prefix="left_" joint_limited="true"/>
   <!-- right arm -->
-  <xacro:ur5_robot prefix="right_" joint_limited="false"/>
+  <xacro:ur5_robot prefix="right_" joint_limited="true"/>
   <link name="world" />
 <!-- box-->
@@ -22,5 +22,5 @@
   <joint name="world_joint" type="fixed">
     <parent link="world" />
-    <child link = "box_link" />
+    <child link="box_link" />
     <origin xyz="0.0 0.0 0.4572" rpy="0.0 0.0 0.0" />
   </joint>
@@ -37,15 +37,20 @@
     <origin xyz="0.762 -0.381 0.4572" rpy="0 0 1.57" />
  </joint>
+ <!-- Force Torque Sensor -->
+ <xacro:include filename="$(find robotiq_force_torque_sensor)/urdf/robotiq_fts300.urdf.xacro" />
+ <xacro:robotiq_fts300 prefix="left_" parent="left_ee_link" >
+   <origin xyz="0.035 0 0.0" rpy="0.0 0 -1.57"/>
+ </xacro:robotiq_fts300>
+ <xacro:robotiq_fts300 prefix="right_" parent="right_ee_link" >
+   <origin xyz="0.035 0 0.0" rpy="0.0 0 -1.57"/>
+ </xacro:robotiq_fts300>
   <!-- GRIPPER -->
   <!-- Import robotiq gazebo and gripper description -->
   <xacro:include filename="$(find robotiq_85_description)/urdf/robotiq_85_gripper.urdf.xacro" />
-  <xacro:robotiq_85_gripper prefix="left_" parent="left_ee_link" >
-        <origin xyz="0 0 0" rpy="0 0 0"/>
-    </xacro:robotiq_85_gripper>
-  <!-- GRIPPER -->
-  <!-- Import robotiq gazebo and gripper description -->
-  <xacro:include filename="$(find robotiq_85_description)/urdf/robotiq_85_gripper.urdf.xacro" />
-  <xacro:robotiq_85_gripper prefix="right_" parent="right_ee_link" >
-        <origin xyz="0 0 0" rpy="0 0 0"/>
-    </xacro:robotiq_85_gripper>
+  <xacro:robotiq_85_gripper prefix="left_" parent="left_fts_toolside" >
+      <origin xyz="0.0 0.0 -0.037" rpy="0.0 0.0 1.57"/>
+  </xacro:robotiq_85_gripper>
+  <xacro:robotiq_85_gripper prefix="right_" parent="right_fts_toolside" >
+      <origin xyz="0.0 0.0 -0.037" rpy="0.0 0.0 1.57"/>
+  </xacro:robotiq_85_gripper>
 </robot>
