Commit message: adjusted to be on either side of the set of tables

File: ur_description/urdf/left_ur5_robotiq_robot_limited.urdf.xacro (robot description, xacro)
@@ -13,10 +13,10 @@
     <visual>
       <geometry>
-        <box size="0.762 1.524 0.9144"/>
+        <box size="2.286 1.524 0.9144"/>
       </geometry>
     </visual>
     <collision>
       <geometry>
-        <box size="0.762 1.524 0.9144"/>
+        <box size="2.286 1.524 0.9144"/>
       </geometry>
     </collision>

File: ur_description/urdf/right_ur5_robotiq_robot_limited.urdf.xacro (robot description, xacro)
@@ -13,10 +13,10 @@
     <visual>
       <geometry>
-        <box size="0.762 1.524 0.9144"/>
+        <box size="2.286 1.524 0.9144"/>
       </geometry>
     </visual>
     <collision>
       <geometry>
-        <box size="0.762 1.524 0.9144"/>
+        <box size="2.286 1.524 0.9144"/>
       </geometry>
     </collision>
@@ -33,9 +33,9 @@
   </joint>
 <!-- attach the robot to the box -->
- <joint name="right_box_joint" type="fixed">
-    <parent link="box_link"/>
-    <child link="right_base_link"/>
-    <origin xyz="0.0 -0.381 0.4572" rpy="0 0 1.57" />
- </joint>
+   <joint name="right_box_joint" type="fixed">
+      <parent link="box_link"/>
+      <child link="right_base_link"/>
+      <origin xyz="0.762 -0.381 0.4572" rpy="0 0 1.57" />
+   </joint>
  <!-- Force Torque Sensor -->
  <xacro:include filename="$(find robotiq_force_torque_sensor)/urdf/robotiq_fts300.urdf.xacro" />

Commit message: updated box position

File: ur_description/urdf/left_ur5_robotiq_robot_limited.urdf.xacro (robot description, xacro)
@@ -33,9 +33,9 @@
   </joint>
 <!-- attach the robot to the box -->
- <joint name="left_box_joint" type="fixed">
-    <parent link="box_link"/>
-    <child link="left_base_link"/>
-    <origin xyz="0.0 -0.381 0.4572" rpy="0 0 1.57" />
- </joint>
+   <joint name="left_box_joint" type="fixed">
+      <parent link="box_link"/>
+      <child link="left_base_link"/>
+      <origin xyz="-0.762 -0.381 0.4572" rpy="0 0 1.57" />
+   </joint>
  <!-- Force Torque Sensor -->
  <xacro:include filename="$(find robotiq_force_torque_sensor)/urdf/robotiq_fts300.urdf.xacro" />
