Commit message: Adding collision and mass information regarding the table

File: ur_description/urdf/ur5_robotiq_robot_limited.urdf.xacro (robot description, xacro)
@@ -16,4 +16,13 @@
       </geometry>
     </visual>
+    <collision>
+      <geometry>
+        <box size="0.762 1.524 0.9144"/>
+      </geometry>
+    </collision>
+    <inertial>
+      <mass value="100"/>
+      <inertia ixx="10" ixy="0.0" ixz="0.0" iyy="10" iyz="0.0" izz="10"/>
+    </inertial>
   </link>
 <!-- attach the box to the world-->

Commit message: Bigger table for running the single robot.

File: ur_description/urdf/ur5_robotiq_robot_limited.urdf.xacro (robot description, xacro)
@@ -13,10 +13,10 @@
     <visual>
       <geometry>
-        <box size="0.762 1.524 0.9144"/>
+        <box size="2.286 1.524 0.9144"/>
       </geometry>
     </visual>
     <collision>
       <geometry>
-        <box size="0.762 1.524 0.9144"/>
+        <box size="2.286 1.524 0.9144"/>
       </geometry>
     </collision>

Commit message: fixing table size

File: ur_description/urdf/ur5_robotiq_robot_limited.urdf.xacro (robot description, xacro)
@@ -13,10 +13,10 @@
     <visual>
       <geometry>
-        <box size="2.286 1.524 0.9144"/>
+        <box size="0.73 1.55 0.9144"/>
       </geometry>
     </visual>
     <collision>
       <geometry>
-        <box size="2.286 1.524 0.9144"/>
+        <box size="2.19 1.55 0.9144"/>
       </geometry>
     </collision>

Commit message: Alternative URDF for the robotiq gripper. All joints are fixed as a temporary solution.

File: ur_description/urdf/ur5_robotiq_robot_limited.urdf.xacro (robot description, xacro)
@@ -45,8 +45,10 @@
  <!-- GRIPPER -->
  <!-- Import robotiq gazebo and gripper description -->
- <xacro:include filename="$(find robotiq_85_description)/urdf/robotiq_85_gripper.urdf.xacro" />
+ <!-- xacro:include filename="$(find robotiq_85_description)/urdf/robotiq_85_gripper.urdf.xacro" /-->
+ <xacro:include filename="$(find robotiq_85_description)/urdf/robotiq_arg85_description.urdf.xacro" />
  <xacro:robotiq_85_gripper prefix="" parent="fts_toolside" >
-       <origin xyz="0.0 0.0 -0.037" rpy="0.0 0.0 1.57"/>
-   </xacro:robotiq_85_gripper>
+   <!-- origin xyz="0.0 0.0 -0.037" rpy="0.0 0.0 1.57"/-->
+   <origin xyz="0.0 0.0 -0.037" rpy="-1.57 3.1415 0.0"/>
+ </xacro:robotiq_85_gripper>
 <!--origin xyz="0.0 0 0.025" rpy="0.0 -1.57 1.57"/-->
 </robot>
