Commit message: added force/torque sensor to urdfs of robots

File: ur_description/urdf/ur5_robotiq85_kinect_table.urdf.xacro (robot description, xacro)
@@ -29,10 +29,15 @@
     <origin xyz="0.0 -0.381 0.4572" rpy="0 0 1.57" />
  </joint>
-  <!-- GRIPPER -->
-  <!-- Import robotiq gazebo and gripper description -->
-  <xacro:include filename="$(find robotiq_85_description)/urdf/robotiq_85_gripper.urdf.xacro" />
-  <xacro:robotiq_85_gripper prefix="" parent="ee_link" >
-        <origin xyz="0 0 0" rpy="0 0 0"/>
-    </xacro:robotiq_85_gripper>
+ <!-- Force Torque Sensor -->
+ <xacro:include filename="$(find robotiq_force_torque_sensor)/urdf/robotiq_fts300.urdf.xacro" />
+ <xacro:robotiq_fts300 prefix="" parent="ee_link" >
+   <origin xyz="0.035 0 0.0" rpy="0.0 0 -1.57"/>
+ </xacro:robotiq_fts300>
+ <!-- GRIPPER -->
+ <!-- Import robotiq gazebo and gripper description -->
+ <xacro:include filename="$(find robotiq_85_description)/urdf/robotiq_85_gripper.urdf.xacro" />
+ <xacro:robotiq_85_gripper prefix="" parent="fts_toolside" >
+       <origin xyz="0.0 0.0 -0.037" rpy="0.0 0.0 1.57"/>
+   </xacro:robotiq_85_gripper>>
  <!--kinect  -->
  <xacro:include filename="$(find ur_description)/urdf/sensors/kinect.urdf.xacro"/>

File: ur_description/urdf/ur5_robotiq_robot.urdf.xacro (robot description, xacro)
@@ -29,9 +29,14 @@
     <origin xyz="0.0 -0.381 0.4572" rpy="0 0 1.57" />
  </joint>
-  <!-- GRIPPER -->
-  <!-- Import robotiq gazebo and gripper description -->
-  <xacro:include filename="$(find robotiq_85_description)/urdf/robotiq_85_gripper.urdf.xacro" />
-  <xacro:robotiq_85_gripper prefix="" parent="ee_link" >
-        <origin xyz="0 0 0" rpy="0 0 0"/>
-    </xacro:robotiq_85_gripper>
+ <!-- Force Torque Sensor -->
+ <xacro:include filename="$(find robotiq_force_torque_sensor)/urdf/robotiq_fts300.urdf.xacro" />
+ <xacro:robotiq_fts300 prefix="" parent="ee_link" >
+   <origin xyz="0.035 0 0.0" rpy="0.0 0 -1.57"/>
+ </xacro:robotiq_fts300>
+ <!-- GRIPPER -->
+ <!-- Import robotiq gazebo and gripper description -->
+ <xacro:include filename="$(find robotiq_85_description)/urdf/robotiq_85_gripper.urdf.xacro" />
+ <xacro:robotiq_85_gripper prefix="" parent="fts_toolside" >
+       <origin xyz="0.0 0.0 -0.037" rpy="0.0 0.0 1.57"/>
+   </xacro:robotiq_85_gripper>
 </robot>

File: ur_description/urdf/ur5_robotiq_robot_limited.urdf.xacro (robot description, xacro)
@@ -29,5 +29,5 @@
   <joint name="world_joint" type="fixed">
     <parent link="world" />
-    <child link = "box_link" />
+    <child link="box_link" />
     <origin xyz="0.0 0.0 0.4572" rpy="0.0 0.0 0.0" />
   </joint>
@@ -38,9 +38,15 @@
     <origin xyz="0.0 -0.381 0.4572" rpy="0 0 1.57" />
  </joint>
-  <!-- GRIPPER -->
-  <!-- Import robotiq gazebo and gripper description -->
-  <xacro:include filename="$(find robotiq_85_description)/urdf/robotiq_85_gripper.urdf.xacro" />
-  <xacro:robotiq_85_gripper prefix="" parent="ee_link" >
-        <origin xyz="0 0 0" rpy="0 0 0"/>
-    </xacro:robotiq_85_gripper>
+ <!-- Force Torque Sensor -->
+ <xacro:include filename="$(find robotiq_force_torque_sensor)/urdf/robotiq_fts300.urdf.xacro" />
+ <xacro:robotiq_fts300 prefix="" parent="ee_link" >
+   <origin xyz="0.035 0 0.0" rpy="0.0 0 -1.57"/>
+ </xacro:robotiq_fts300>
+ <!-- GRIPPER -->
+ <!-- Import robotiq gazebo and gripper description -->
+ <xacro:include filename="$(find robotiq_85_description)/urdf/robotiq_85_gripper.urdf.xacro" />
+ <xacro:robotiq_85_gripper prefix="" parent="fts_toolside" >
+       <origin xyz="0.0 0.0 -0.037" rpy="0.0 0.0 1.57"/>
+   </xacro:robotiq_85_gripper>
+<!--origin xyz="0.0 0 0.025" rpy="0.0 -1.57 1.57"/-->
 </robot>

Commit message: Support for limited joint angles
The planner fails at every attempt tested. Joint limits were added
to this configuration but the planner still fails.

File: ur_description/urdf/ur5_robotiq85_kinect_table.urdf.xacro (robot description, xacro)
@@ -2,4 +2,5 @@
 <robot xmlns:xacro="http://ros.org/wiki/xacro"
        name="ur5_robotiq85_kinect" >
+  <xacro:arg name="limited" default="false"/>
   <!-- common stuff -->
   <xacro:include filename="$(find ur_description)/urdf/common.gazebo.xacro" />
@@ -7,7 +8,7 @@
   <xacro:include filename="$(find ur_description)/urdf/ur5.urdf.xacro" />
   <!-- arm -->
-  <xacro:ur5_robot prefix="" joint_limited="false"/>
+  <xacro:ur5_robot prefix="" joint_limited="$(arg limited)"/>
   <link name="world" />
-<!-- box-->
+  <!-- box-->
   <link name="box_link">
     <visual>
@@ -16,4 +17,13 @@
       </geometry>
     </visual>
+    <collision>
+      <geometry>
+        <box size="0.762 1.524 0.9144"/>
+      </geometry>
+    </collision>
+    <inertial>
+      <mass value="100"/>
+      <inertia ixx="10" ixy="0.0" ixz="0.0" iyy="10" iyz="0.0" izz="10"/>
+    </inertial>
   </link>
 <!-- attach the box to the world-->
