Commit message: Changes for Kinetic and our setup

File: ur_description/urdf/ur5.urdf.xacro (robot description, xacro)
@@ -39,4 +39,5 @@
   <xacro:property name="shoulder_offset" value="0.13585" />  <!-- measured from model -->
   <xacro:property name="elbow_offset" value="-0.1197" /> <!-- measured from model -->
+  <xacro:property name="angle_offset" value="${pi * 0.5}" /> <!-- measured from model -->
   <!-- link lengths used in model -->
   <xacro:property name="shoulder_height" value="${ur5_d1}" />
@@ -90,5 +91,5 @@
       <parent link="${prefix}base_link" />
       <child link = "${prefix}shoulder_link" />
-      <origin xyz="0.0 0.0 ${shoulder_height}" rpy="0.0 0.0 0.0" />
+      <origin xyz="0.0 0.0 ${shoulder_height}" rpy="0 0.0 0" />
       <axis xyz="0 0 1" />
       <xacro:unless value="${joint_limited}">
@@ -121,5 +122,6 @@
       <parent link="${prefix}shoulder_link" />
       <child link = "${prefix}upper_arm_link" />
-      <origin xyz="0.0 ${shoulder_offset} 0.0" rpy="0.0 ${pi / 2.0} 0.0" />
+      <origin xyz="0.0 ${shoulder_offset} 0.0" rpy="0.0 ${angle_offset} 0.0" />
+<!--      <origin xyz="0.0 ${shoulder_offset} 0.0" rpy="0.0 ${angle_offset} 0.0" /> -->
       <axis xyz="0 1 0" />
       <xacro:unless value="${joint_limited}">

Commit message: Updated UR5 control framework in simulation to play with the learning framework

File: ur_description/urdf/ur5.urdf.xacro (robot description, xacro)
@@ -39,5 +39,5 @@
   <xacro:property name="shoulder_offset" value="0.13585" />  <!-- measured from model -->
   <xacro:property name="elbow_offset" value="-0.1197" /> <!-- measured from model -->
-  <xacro:property name="angle_offset" value="${pi * 0.5}" /> <!-- measured from model -->
+  <xacro:property name="angle_offset" value="${0}" /> <!-- measured from model -->
   <!-- link lengths used in model -->
   <xacro:property name="shoulder_height" value="${ur5_d1}" />

File: ur_description/urdf/ur5_robot.urdf.xacro (robot description, xacro)
@@ -3,5 +3,5 @@
        name="ur5" >
   <!-- common stuff -->
-  <xacro:include filename="$(find ur_description)/urdf/common.gazebo.xacro" />
+  <!-- <xacro:include filename="$(find ur_description)/urdf/common.gazebo.xacro" /> -->
   <!-- ur5 -->
   <xacro:include filename="$(find ur_description)/urdf/ur5.urdf.xacro" />
@@ -14,3 +14,7 @@
     <origin xyz="0.0 0.0 0.0" rpy="0.0 0.0 0.0" />
   </joint>
+  <gazebo>
+    <plugin name="fetch_gazebo_plugin" filename="libfetch_gazebo_plugin.so"/>
+    <self_collide>1</self_collide>
+  </gazebo>
 </robot>

Commit message: Adedd cable snake models to the meshes, and made the root ur5 urdf use the snake models.

File: ur_description/urdf/ur5.urdf.xacro (robot description, xacro)
@@ -136,13 +136,13 @@
       <visual>
         <geometry>
-          <mesh filename="package://ur_description/meshes/ur5/visual/upperarm.dae" />
-        </geometry>
-        <material name="LightGrey">
-          <color rgba="0.7 0.7 0.7 1.0"/>
-        </material>
-      </visual>
-      <collision>
-        <geometry>
-          <mesh filename="package://ur_description/meshes/ur5/collision/upperarm.stl" />
+          <mesh filename="package://ur_description/meshes/ur5/visual/upperarm_snake.dae" />
+        </geometry>
+        <material name="LightGrey">
+          <color rgba="0.7 0.7 0.7 1.0"/>
+        </material>
+      </visual>
+      <collision>
+        <geometry>
+          <mesh filename="package://ur_description/meshes/ur5/collision/upperarm_snake.stl" />
         </geometry>
       </collision>
@@ -167,13 +167,13 @@
       <visual>
         <geometry>
-          <mesh filename="package://ur_description/meshes/ur5/visual/forearm.dae" />
-        </geometry>
-        <material name="LightGrey">
-          <color rgba="0.7 0.7 0.7 1.0"/>
-        </material>
-      </visual>
-      <collision>
-        <geometry>
-          <mesh filename="package://ur_description/meshes/ur5/collision/forearm.stl" />
+          <mesh filename="package://ur_description/meshes/ur5/visual/forearm_snake.dae" />
+        </geometry>
+        <material name="LightGrey">
+          <color rgba="0.7 0.7 0.7 1.0"/>
+        </material>
+      </visual>
+      <collision>
+        <geometry>
+          <mesh filename="package://ur_description/meshes/ur5/collision/forearm_snake.stl" />
         </geometry>
       </collision>

Commit message: Can see spheres for double ur, removed prefix from controllers, removed dup pi definitions.

File: ur_description/urdf/ur5.urdf.xacro (robot description, xacro)
@@ -3,5 +3,4 @@
   <xacro:include filename="ur.transmission.xacro" />
   <xacro:include filename="ur.gazebo.xacro" />
-  <xacro:property name="pi" value="3.14159265" />
   <!-- Inertia parameters -->
   <xacro:property name="base_mass" value="4.0" />  <!-- This mass might be incorrect -->

Commit message: hardware transmission param for xacro

File: ur_description/urdf/ur5.urdf.xacro (robot description, xacro)
@@ -1,4 +1,5 @@
 <?xml version="1.0"?>
 <robot xmlns:xacro="http://ros.org/wiki/xacro">
+  <xacro:property name="transmission_hw_interface" default="hardware_interface/PositionJointInterface"/>
   <xacro:include filename="ur.transmission.xacro" />
   <xacro:include filename="ur.gazebo.xacro" />
@@ -288,5 +289,5 @@
       </collision>
     </link>
-    <xacro:ur_arm_transmission prefix="${prefix}" />
+    <xacro:ur_arm_transmission prefix="${prefix}" hw_interface="${transmission_hw_interface}" />
     <xacro:ur_arm_gazebo prefix="${prefix}" />
     <!-- ROS base_link to UR 'Base' Coordinates transform -->
