Commit message: Changing the orientation of the depth camera

File: ur_description/urdf/sensors/kinect.urdf.xacro (robot description, xacro)
@@ -4,4 +4,5 @@
   <xacro:include filename="$(find ur_description)/urdf/sensors/kinect_properties.urdf.xacro"/>
   <xacro:macro name="sensor_kinect" params="parent">
+    <link name="camera_rgb_frame"/>
     <joint name="camera_rgb_joint" type="fixed">
       <origin xyz="${cam_px} ${cam_py} ${cam_pz}" rpy="${cam_or} ${cam_op} ${cam_oy}"/>
@@ -9,5 +10,5 @@
       <child link="camera_rgb_frame" />
     </joint>
-    <link name="camera_rgb_frame"/>
+    <link name="camera_rgb_optical_frame"/>
     <joint name="camera_rgb_optical_joint" type="fixed">
       <origin xyz="0 0 0" rpy="${-M_PI/2} 0 ${-M_PI/2}" />
@@ -15,11 +16,5 @@
       <child link="camera_rgb_optical_frame" />
     </joint>
-    <link name="camera_rgb_optical_frame"/>
-    <joint name="camera_joint" type="fixed">
-      <origin xyz="0 ${-cam_py} 0" rpy="0 0 0"/>
-      <parent link="camera_rgb_frame"/>
-      <child link="camera_link"/>
-    </joint>
-      <link name="camera_link">
+  <link name="camera_link">
       <visual>
        <origin xyz="0 0 0" rpy="0 0 ${M_PI/2}"/>
@@ -42,13 +37,21 @@
       </inertial>
     </link>
+    <joint name="camera_joint" type="fixed">
+      <!-- <origin xyz="0 ${-cam_py} 0" rpy="0 0 0"/> -->
+      <origin xyz="0 0 0" rpy="0 0 0"/>
+      <parent link="camera_rgb_frame"/>
+      <child link="camera_link"/>
+    </joint>
     <!-- The fixed joints & links below are usually published by static_transformers launched by the OpenNi launch
          files. However, for Gazebo simulation we need them, so we add them here.
          (Hence, don't publish them additionally!) -->
+  <link name="camera_depth_frame"/>
 	<joint name="camera_depth_joint" type="fixed">
-	  <origin xyz="0 ${-cam_py} 0" rpy="0 0 0" />
+	  <!-- <origin xyz="0 ${-cam_py} 0" rpy="0 0 0" /> -->
+    <origin xyz="0 0 0" rpy="0 0 0" />
 	  <parent link="camera_rgb_frame" />
 	  <child link="camera_depth_frame" />
 	</joint>
-	<link name="camera_depth_frame"/>
+  <link name="camera_depth_optical_frame"/>
 	<joint name="camera_depth_optical_joint" type="fixed">
 	  <origin xyz="0 0 0" rpy="${-M_PI/2} 0 ${-M_PI/2}" />
@@ -56,5 +59,4 @@
 	  <child link="camera_depth_optical_frame" />
 	</joint>
-	<link name="camera_depth_optical_frame"/>
 	<!-- Kinect sensor for simulation -->
 	<ur5_sim_3dsensor/>

File: ur_description/urdf/sensors/kinect_properties.urdf.xacro (robot description, xacro)
@@ -19,10 +19,10 @@
      (currently in development and awaiting feedback)
    -->
-	<xacro:property name="cam_px" value="0" />
-	<xacro:property name="cam_py" value="-0.5" />
-	<xacro:property name="cam_pz" value="0.5" />
+  <xacro:property name="cam_px" value="0" />
+	<xacro:property name="cam_py" value="-0.7" />
+	<xacro:property name="cam_pz" value="0.9" />
 	<xacro:property name="cam_or" value="0" />
-	<xacro:property name="cam_op" value="0.6" />
-	<xacro:property name="cam_oy" value="${M_PI/2}" />
+	<xacro:property name="cam_op" value="${M_PI/4.0}" />
+	<xacro:property name="cam_oy" value="${M_PI/5.0}" />
 	<xacro:property name="M_PI" value="3.1415926535897931" />
 </robot>

File: ur_description/urdf/ur5_robotiq_robot_limited.urdf.xacro (robot description, xacro)
@@ -13,10 +13,10 @@
     <visual>
       <geometry>
-        <box size="0.762 1.524 0.9144"/>
+        <box size="3 3 0.9144"/>
       </geometry>
     </visual>
     <collision>
       <geometry>
-        <box size="0.762 1.524 0.9144"/>
+        <box size="3 3 0.9144"/>
       </geometry>
     </collision>
@@ -36,5 +36,5 @@
     <parent link="box_link"/>
     <child link="base_link"/>
-    <origin xyz="0.0 -0.381 0.4572" rpy="0 0 1.57" />
+    <origin xyz="0.0 -1.2 0.4572" rpy="0 0 1.57" />
  </joint>
  <!-- Force Torque Sensor -->
@@ -50,3 +50,7 @@
    </xacro:robotiq_85_gripper>
 <!--origin xyz="0.0 0 0.025" rpy="0.0 -1.57 1.57"/-->
+  <!--kinect  -->
+  <xacro:include filename="$(find ur_description)/urdf/sensors/kinect.urdf.xacro"/>
+  <!--attach the kinect to the robot -->
+  <xacro:sensor_kinect  parent="base_link"/>
 </robot>
