Commit message: Changed position of camera to better detect grasps

File: ur_description/urdf/sensors/kinect_properties.urdf.xacro (robot description, xacro)
@@ -19,10 +19,16 @@
      (currently in development and awaiting feedback)
    -->
-  <xacro:property name="cam_px" value="0" />
-	<xacro:property name="cam_py" value="-0.7" />
+  <!-- <xacro:property name="cam_px" value="0.05" />
+	<xacro:property name="cam_py" value="-0.75" />
 	<xacro:property name="cam_pz" value="0.9" />
 	<xacro:property name="cam_or" value="0" />
 	<xacro:property name="cam_op" value="${M_PI/4.0}" />
-	<xacro:property name="cam_oy" value="${M_PI/5.0}" />
+	<xacro:property name="cam_oy" value="${M_PI/5.0}" /> -->
+  <xacro:property name="cam_px" value="0.15" />
+	<xacro:property name="cam_py" value="0" />
+	<xacro:property name="cam_pz" value="0.04" />
+	<xacro:property name="cam_or" value="0" />
+	<xacro:property name="cam_op" value="0" />
+	<xacro:property name="cam_oy" value="0" />
 	<xacro:property name="M_PI" value="3.1415926535897931" />
 </robot>

File: ur_description/urdf/ur5_robotiq_robot_limited.urdf.xacro (robot description, xacro)
@@ -15,4 +15,7 @@
         <box size="3 3 0.9144"/>
       </geometry>
+      <material name="white">
+        <color rgba="1 1 1 1"/>
+      </material>
     </visual>
     <collision>

Commit message: change camera location

File: ur_description/urdf/sensors/kinect_properties.urdf.xacro (robot description, xacro)
@@ -19,12 +19,12 @@
      (currently in development and awaiting feedback)
    -->
-  <!-- <xacro:property name="cam_px" value="0.05" />
-	<xacro:property name="cam_py" value="-0.75" />
-	<xacro:property name="cam_pz" value="0.9" />
+  <!-- <xacro:property name="cam_px" value="0.15" />
+	<xacro:property name="cam_py" value="0" />
+	<xacro:property name="cam_pz" value="0.04" />
 	<xacro:property name="cam_or" value="0" />
-	<xacro:property name="cam_op" value="${M_PI/4.0}" />
-	<xacro:property name="cam_oy" value="${M_PI/5.0}" /> -->
-  <xacro:property name="cam_px" value="0.15" />
-	<xacro:property name="cam_py" value="0" />
+	<xacro:property name="cam_op" value="0" />
+	<xacro:property name="cam_oy" value="0" /> -->
+  <xacro:property name="cam_px" value="0.0" />
+	<xacro:property name="cam_py" value="-0.25" />
 	<xacro:property name="cam_pz" value="0.04" />
 	<xacro:property name="cam_or" value="0" />
